File: pcb/pcb.kicad_pcb (KiCad board)
At the start: 2 copper layers, 120.6 x 167.6 mm, 32 parts, among them J1 Screw_Terminal_01x02, U1 L293D

Commit message: WIP async and new pcb layout
Parts:
- MF1, MF2: footprint pcb:motorized_fader -> Quint:motorized_fader
- U1: value L293D -> Pololu_Breakout_DRV8833; footprint Package_DIP:DIP-16_W7.62mm -> Quint:Pololu_DRV8833
- moved U1 24.5 mm to (96.5, 63.5), turned to -90 degrees
- moved MF2 3.62 mm to (54.8, 101.6)
- moved MF1 0.12 mm to (35.7, 101.6)
Connections:
- MF1 pad 1: fader1 -> +5V
- MF1 pad 2: +5V -> fader1
- MF1 pad 3: Net-(MF1-Pad3) -> Earth
- MF1 pad 4: Net-(MF1-Pad4) -> unconnected-(MF1-Pad4)
- MF1 pad 5: Net-(MF1-Pad5) -> unconnected-(MF1-Pad5)
- MF2 pad 1: fader2 -> +5V
- MF2 pad 2: +5V -> fader2
- MF2 pad 3: Net-(MF2-Pad3) -> Earth
- MF2 pad 4: Net-(MF2-Pad4) -> unconnected-(MF2-Pad4)
- MF2 pad 5: Net-(MF2-Pad5) -> unconnected-(MF2-Pad5)
- PM1 pad 14: Net-(PM1-Pad14) -> unconnected-(PM1-Pad14)
- PM1 pad 15: Net-(PM1-Pad15) -> unconnected-(PM1-Pad15)
- PM1 pad 2: Net-(PM1-Pad2) -> unconnected-(PM1-Pad2)
- PM1 pad 3: Net-(PM1-Pad3) -> unconnected-(PM1-Pad3)
- U1 pad 1: +5V -> unconnected-(U1-Pad1)
- U1 pad 10: M2_pos -> Net-(MF2-Pad6)
- U1 pad 11: Net-(MF2-Pad6) -> Net-(MF2-Pad7)
- U1 pad 12: Earth -> Net-(MF1-Pad7)
- U1 pad 13: Earth -> Net-(MF1-Pad6)
- U1 pad 14: Net-(MF2-Pad7) -> unconnected-(U1-Pad14)
- U1 pad 15: M2_neg -> unconnected-(U1-Pad15)
- U1 pad 2: M1_pos -> M2_pos
- U1 pad 3: Net-(MF1-Pad7) -> M2_neg
- U1 pad 4: Earth -> M1_pos
- U1 pad 5: Earth -> M1_neg
- U1 pad 6: Net-(MF1-Pad6) -> unconnected-(U1-Pad6)
- U1 pad 7: M1_neg -> unconnected-(U1-Pad7)
- U1 pad 8: +5V -> Earth
Routing:
- net Earth: track 76.1 -> 159.0 mm, vias 1 -> 0
- net fader1: track 61.4 -> 86.3 mm
- net M1_pos: track 48.1 -> 30.8 mm
- net fader2: track 36.5 -> 53.6 mm
- net +5V: track 223.4 -> 236.6 mm
- net Net-(MF2-Pad6): track 85.0 -> 72.9 mm
- net Net-(MF1-Pad7): track 78.3 -> 89.6 mm
- net Net-(MF2-Pad7): track 86.1 -> 75.2 mm
- net M1_neg: track 41.8 -> 31.2 mm
- net M2_neg: track 24.4 -> 14.5 mm
- net M2_pos: track 30.6 -> 22.1 mm
- net fader_cap2: track 68.1 -> 70.5 mm
- net fader_cap1: track 74.1 -> 75.1 mm
- net Net-(MF1-Pad6): track 78.3 -> 77.7 mm
- removed copper zone on F.Cu, net Earth
Other:
- net class Default removed
